Commit message: Update rover.urdf.xacro

File: rover_description/urdf/rover.urdf.xacro (robot description, xacro)
@@ -1,560 +1,181 @@
 <?xml version="1.0"?>
-<robot xmlns:xacro="http://ros.org/wiki/xacro"
-       name="mars_opportunity_rover">
-  <!-- ========================================================= -->
-  <!-- Global Parameters -->
-  <!-- ========================================================= -->
-  <xacro:property name="chassis_length" value="0.75"/>
-  <xacro:property name="chassis_width" value="0.45"/>
-  <xacro:property name="chassis_height" value="0.20"/>
-  <xacro:property name="chassis_mass" value="12.0"/>
-  <xacro:property name="wheel_radius"  value="0.065"/>
-  <xacro:property name="wheel_width"  value="0.025"/>
-  <xacro:property name="wheel_mass"  value="1.2"/>
-  <xacro:property name="arm_l1"  value="0.12"/>
-  <xacro:property name="arm_l2"  value="0.18"/>
-  <xacro:property name="arm_l3"  value="0.20"/>
-  <xacro:property name="arm_l4"  value="0.15"/>
-  <xacro:property name="arm_l5"  value="0.07"/>
-  <xacro:property name="arm_radius"  value="0.025"/>
-  <xacro:property name="arm_link_mass"  value="1.0"/>
-  <xacro:property name="scale_x"  value="0.68"/>
-  <xacro:property name="scale_y"  value="0.68"/>
-  <xacro:property name="scale_z"  value="0.68"/>
-  <!-- ================= Mesh Path Parameters ================== -->
-  <!-- Mesh Path Parameters - Chassis -->
-  <xacro:property name="chassis_mesh_0" value="package://rover_description/meshes/mesh_0.stl"/>
-  <xacro:property name="wheel_mesh"  value=""/>
-  <!-- Mesh Path Parameters - Head -->
-  <xacro:property name="head_base_mesh_2" value="package://rover_description/meshes/mesh_2.stl"/>
-  <xacro:property name="head_top_mesh_3" value="package://rover_description/meshes/mesh_3.stl"/>
-  <!-- Mesh Path Parameters - Solar Panels -->
-  <xacro:property name="panel_left_front_mesh_5" value="package://rover_description/meshes/mesh_5.stl"/>
-  <xacro:property name="panel_left_rear_mesh_6" value="package://rover_description/meshes/mesh_6.stl"/>
-  <xacro:property name="panel_right_front_mesh_7" value="package://rover_description/meshes/mesh_7.stl"/>
-  <xacro:property name="panel_right_rear_mesh_8" value="package://rover_description/meshes/mesh_8.stl"/>
-  <xacro:property name="panel_center_rear_mesh_9" value="package://rover_description/meshes/mesh_9.stl"/>
-  <!-- Mesh Path Parameters - Robotic Arm -->
-  <xacro:property name="arm_base_mesh_60"  value="ackage://rover_description/meshes/mesh_60.stl"/>
-  <xacro:property name="arm_l1_mesh_61"  value="package://rover_description/meshes/mesh_61.stl"/>
-  <xacro:property name="arm_l2_mesh_62"  value="package://rover_description/meshes/mesh_62.stl"/>
-  <xacro:property name="arm_l3_mesh_63"  value="package://rover_description/meshes/mesh_63.stl"/>
-  <xacro:property name="arm_l4_mesh_64"  value="package://rover_description/meshes/mesh_64.stl"/>
-  <xacro:property name="arm_l5_mesh_65"   value="package://rover_description/meshes/mesh_65.stl"/>
-  <xacro:property name="arm_head_mesh_66"  value="package://rover_description/meshes/mesh_66.stl"/>
-  <xacro:property name="arm_tools_mesh_67"  value="package://rover_description/meshes/mesh_67.stl"/>
-  <!-- Mesh Path Parameters - Group Steering Left -->
-  <xacro:property name="group_left_chassis_joint_mesh_10"  value="package://rover_description/meshes/mesh_10.stl"/>
-  <xacro:property name="group_left_front_suspension_mesh_11"  value="package://rover_description/meshes/mesh_11.stl"/>
-  <xacro:property name="group_left_front_steering_mesh_12"  value="package://rover_description/meshes/mesh_12.stl"/>
-  <xacro:property name="group_left_front_wheel_mesh_13"  value="package://rover_description/meshes/mesh_13.stl"/>
-  <xacro:property name="group_left_middle_suspension_mesh_14"  value="package://rover_description/meshes/mesh_14.stl"/>
-  <xacro:property name="group_left_middle_chariot_joint_mesh_15"  value="package://rover_description/meshes/mesh_15.stl"/>
-  <xacro:property name="group_left_middle_chariot_center_mesh_16"  value="package://rover_description/meshes/mesh_16.stl"/>
-  <xacro:property name="group_left_middle_chariot_center_wheel_mesh_17"  value="package://rover_description/meshes/mesh_17.stl"/>
-  <xacro:property name="group_left_middle_chariot_rear_mesh_18"  value="package://rover_description/meshes/mesh_18.stl"/>
-  <xacro:property name="group_left_middle_chariot_steering_mesh_19"  value="package://rover_description/meshes/mesh_19.stl"/>
-  <xacro:property name="group_left_middle_chariot_wheel_mesh_20"  value="package://rover_description/meshes/mesh_20.stl"/>
-  <!-- Mesh Path Parameters - Group Steering Right -->
-  <xacro:property name="group_right_chassis_joint_mesh_30"  value="package://rover_description/meshes/mesh_30.stl"/>
-  <xacro:property name="group_right_front_suspension_mesh_31"  value="package://rover_description/meshes/mesh_31.stl"/>
-  <xacro:property name="group_right_front_steering_mesh_32"  value="package://rover_description/meshes/mesh_32.stl"/>
-  <xacro:property name="group_right_front_wheel_mesh_33"  value="package://rover_description/meshes/mesh_33.stl"/>
-  <xacro:property name="group_right_middle_suspension_mesh_34"  value="package://rover_description/meshes/mesh_34.stl"/>
-  <xacro:property name="group_right_middle_chariot_joint_mesh_35"  value="package://rover_description/meshes/mesh_35.stl"/>
-  <xacro:property name="group_right_middle_chariot_center_mesh_36"  value="package://rover_description/meshes/mesh_36.stl"/>
-  <xacro:property name="group_right_middle_chariot_center_wheel_mesh_37"  value="package://rover_description/meshes/mesh_37.stl"/>
-  <xacro:property name="group_right_middle_chariot_rear_mesh_38"  value="package://rover_description/meshes/mesh_38.stl"/>
-  <xacro:property name="group_right_middle_chariot_steering_mesh_39"  value="package://rover_description/meshes/mesh_39.stl"/>
-  <xacro:property name="group_right_middle_chariot_wheel_mesh_40"  value="package://rover_description/meshes/mesh_40.stl"/>
-  <!-- Mesh Path Parameters - Antenna High Gain-->
-  <xacro:property name="antenna_base_mesh_70"  value="package://rover_description/meshes/mesh_70.stl"/>
-  <xacro:property name="antenna_top_mesh_71"  value="package://rover_description/meshes/mesh_71.stl"/>
+<!-- rover_full.urdf.xacro
+     Six-wheeled rover: 6 wheels (FL, ML, RL on left and FR, MR, RR on right)
+     Four steering joints: FL, FR, RL, RR (corner servos)
+     5-DOF arm mounted at front center
+     - All key dimensions are parameters at the top for easy tuning.
+     - Includes transmissions suitable for ros_control (velocity for wheels, position for steering, position/trajectory for arm).
+     - Basic Gazebo plugin placeholders for imu, kinect (rgbd), and gps.
+-->
+<robot xmlns:xacro="http://www.ros.org/wiki/xacro" name="six_wheel_rover">
+  <!-- ============================
+       USER-TUNABLE PARAMETERS
+       Edit these values to match your hardware
+       ============================ -->
+  <xacro:property name="wheel_radius" value="0.08"/>        <!-- meters -->
+  <xacro:property name="wheel_thickness" value="0.04"/>
+  <xacro:property name="track" value="0.7"/>               <!-- distance between left & right -->
+  <xacro:property name="half_track" value="${track/2.0}"/>
+  <xacro:property name="front_axle_x" value="0.45"/>
+  <xacro:property name="mid_axle_x" value="0.0"/>
+  <xacro:property name="rear_axle_x" value="-0.45"/>
+  <xacro:property name="base_length" value="0.9"/>
+  <xacro:property name="base_width" value="${track}"/>
+  <xacro:property name="base_height" value="0.18"/>
+  <xacro:property name="wheel_mass" value="0.8"/>
+  <xacro:property name="body_mass" value="25.0"/>
+  <xacro:property name="steer_servo_mass" value="0.3"/>
+  <!-- Arm parameters (5-DOF) -->
+  <xacro:property name="arm_base_height" value="0.20"/>
+  <xacro:property name="arm_link1_len" value="0.10"/>
+  <xacro:property name="arm_link2_len" value="0.18"/>
+  <xacro:property name="arm_link3_len" value="0.16"/>
+  <xacro:property name="arm_link4_len" value="0.12"/>
+  <xacro:property name="arm_link5_len" value="0.08"/>
+  <xacro:property name="arm_joint_limits" value="{'j1':3.14,'j2':1.6,'j3':1.6,'j4':3.14,'j5':3.14}"/>
   <!-- Misc -->
   <xacro:property name="encoder_cpr" value="1024"/>  <!-- counts per rev -->
   <xacro:property name="wheel_inertia" value="0.02"/>
   <xacro:property name="frame_prefix" value=""/>     <!-- set if you want a prefix for joint/link names -->
-  <!-- ========================================================= -->
-  <!-- Base Chassis with Mesh -->
-  <!-- ========================================================= -->
-  <!-- The base link  -  the reference link for the entire model -->
-  <link name="base_link">
-    <visual>
-      <origin xyz="0 0 ${chassis_height/2.0}" rpy="0 0 0"/>
-      <geometry>
-        <mesh filename="${chassis_mesh_0}" scale="${scale_x} ${scale_y} ${scale_z}"/>
-      </geometry>
+  <!-- Helper macro: simple inertia for a box -->
+  <xacro:macro name="box_inertial" params="m lx ly lz">
+    <inertial>
+      <mass value="${m}"/>
+      <origin xyz="0 0 0"/>
+      <inertia ixx="${m*(ly*ly + lz*lz)/12.0}" ixy="0.0" ixz="0.0"
+               iyy="${m*(lx*lx + lz*lz)/12.0}" iyz="0.0"
+               izz="${m*(lx*lx + ly*ly)/12.0}"/>
+    </inertial>
+  </xacro:macro>
+  <!-- ========= base link ========= -->
+  <link name="${frame_prefix}base_link">
+    <visual>
+      <origin xyz="0 0 ${base_height/2.0}" rpy="0 0 0"/>
+      <geometry>
+        <box size="${base_length} ${base_width} ${base_height}"/>
+      </geometry>
+      <material name="blue"/>
     </visual>
     <collision>
-      <origin xyz="0 0 ${chassis_height/2.0}" rpy="0 0 0"/>
-      <geometry>
-        <box size="${chassis_length} ${chassis_width} ${chassis_height}"/>
+      <origin xyz="0 0 ${base_height/2.0}" rpy="0 0 0"/>
+      <geometry>
+        <box size="${base_length} ${base_width} ${base_height}"/>
       </geometry>
     </collision>
+    <!-- inertial -->
+    <xacro:box_inertial m="${body_mass}" lx="${base_length}" ly="${base_width}" lz="${base_height}"/>
+  </link>
+  <!-- ========= helper: wheel model ========= -->
+  <xacro:macro name="wheel" params="side name x y">
+    <link name="${frame_prefix}${name}_wheel_link">
+      <visual>
+        <origin xyz="0 0 0" rpy="0 0 0"/>
+        <geometry>
+          <cylinder length="${wheel_thickness}" radius="${wheel_radius}"/>
+        </geometry>
+      </visual>
+      <collision>
+        <origin xyz="0 0 0" rpy="0 0 0"/>
+        <geometry>
+          <cylinder length="${wheel_thickness}" radius="${wheel_radius}"/>
+        </geometry>
+      </collision>
+      <inertial>
+        <mass value="${wheel_mass}"/>
+        <origin xyz="0 0 0"/>
+        <inertia ixx="${wheel_inertia}" ixy="0" ixz="0" iyy="${wheel_inertia}" iyz="0" izz="${wheel_inertia}"/>
+      </inertial>
+    </link>
+    <!-- wheel revolute joint (rotation axis Y for rolling) -->
+    <joint name="${frame_prefix}${name}_wheel_joint" type="continuous">
+      <parent link="${frame_prefix}${side}_steer_link"/>
+      <child link="${frame_prefix}${name}_wheel_link"/>
+      <!-- wheel is located at x,y relative to steer link's origin -->
+      <origin xyz="${x} ${y} 0" rpy="0 0 0"/>
+      <axis xyz="0 1 0"/>
+    </joint>
+  </xacro:macro>
+  <!-- ========= helper: steer block ========= -->
+  <xacro:macro name="steer_block" params="side steer_name steer_joint_x steer_joint_y">
+    <link name="${frame_prefix}${side}_steer_link">
+      <visual>
+        <origin xyz="0 0 0" rpy="0 0 0"/>
+        <geometry>
+          <box size="0.06 0.08 0.06"/>
+        </geometry>
+      </visual>
+      <collision>
+        <origin xyz="0 0 0" rpy="0 0 0"/>
+        <geometry>
+          <box size="0.06 0.08 0.06"/>
+        </geometry>
+      </collision>
+      <inertial>
+        <mass value="${steer_servo_mass}"/>
+        <origin xyz="0 0 0"/>
+        <inertia ixx="0.001" ixy="0.0" ixz="0.0" iyy="0.001" iyz="0.0" izz="0.001"/>
+      </inertial>
+    </link>
+    <joint name="${frame_prefix}${side}_steer_joint" type="continuous">
+      <parent link="${frame_prefix}base_link"/>
+      <child link="${frame_prefix}${side}_steer_link"/>
+      <origin xyz="${steer_joint_x} ${steer_joint_y} 0" rpy="0 0 0"/>
+      <axis xyz="0 0 1"/>
+    </joint>
+  </xacro:macro>
+  <!-- ========= instantiate steer blocks and wheels ========= -->
+  <!-- Left front -->
+  <xacro:steer_block side="fl" steer_name="fl_steer" steer_joint_x="${front_axle_x}" steer_joint_y="${half_track}"/>
+  <xacro:wheel side="fl" name="fl" x="0 0 0" y="0"/>
+  <!-- Left middle (no steer, attach directly to base_link) -->
+  <link name="${frame_prefix}ml_steer_link">
+    <visual>
+      <origin xyz="0 0 0" rpy="0 0 0"/>
+      <geometry>
+        <box size="0.02 0.02 0.02"/>
+      </geometry>
+    </visual>
     <inertial>
-      <mass value="${chassis_mass}"/>
+      <mass value="0.05"/>
       <origin xyz="0 0 0"/>
-      <inertia ixx="1.0" iyy="1.0" izz="1.0"/>
+      <inertia ixx="1e-4" ixy="0" ixz="0" iyy="1e-4" iyz="0" izz="1e-4"/>
     </inertial>
   </link>
-  <!-- Head -->
-  <joint name="head_base_joint" type="fixed">
-    <parent link="base_link"/>
-    <child  link="head_base_link"/>
-    <origin xyz="0.24 0 0.14" rpy="0 0 0"/>
-    <limit lower="0" upper="0" effort="0" velocity="1.0"/>
-  </joint>
-  <link name="head_base_link">
+  <joint name="${frame_prefix}ml_mount_joint" type="fixed">
+    <parent link="${frame_prefix}base_link"/>
+    <child link="${frame_prefix}ml_steer_link"/>
+    <origin xyz="${mid_axle_x} ${half_track} 0" rpy="0 0 0"/>
+  </joint>
+  <xacro:wheel side="ml" name="ml" x="0 0 0" y="0"/>
+  <!-- Left rear -->
+  <xacro:steer_block side="rl" steer_name="rl_steer" steer_joint_x="${rear_axle_x}" steer_joint_y="${half_track}"/>
+  <xacro:wheel side="rl" name="rl" x="0 0 0" y="0"/>
+  <!-- Right side: mirror y coordinate to -half_track -->
+  <xacro:steer_block side="fr" steer_name="fr_steer" steer_joint_x="${front_axle_x}" steer_joint_y="${-half_track}"/>
+  <xacro:wheel side="fr" name="fr" x="0 0 0" y="0"/>
+  <link name="${frame_prefix}mr_steer_link">
     <visual>
       <origin xyz="0 0 0" rpy="0 0 0"/>
       <geometry>
-        <mesh filename="${head_base_mesh_2}" scale="${scale_x} ${scale_y} ${scale_z}"/>
-      </geometry>
-      <material name="head_base_material"/>
-    </visual>
-    <collision>
-      <origin xyz="0 0 0" rpy="0 0 0"/>
-      <geometry><mesh filename="${head_base_mesh_2}"/></geometry>
-    </collision>
-  </link>
-  <joint name="head_top_joint" type="fixed">
-    <parent link="head_base_link"/>
-    <child  link="head_top_link"/>
-    <origin xyz="0 -0.012 0.33" rpy="0 0 0"/>
-    <limit lower="0" upper="0" effort="0" velocity="1.0"/>
-  </joint>
-  <link name="head_top_link">
-    <visual>
-      <origin xyz="0 0 0" rpy="0 0 0"/>
-      <geometry>
-        <mesh filename="${head_top_mesh_3}" scale="${scale_x} ${scale_y} ${scale_z}"/>
-      </geometry>
-      <material name="head_top_material"/>
-    </visual>
-    <collision>
-      <origin xyz="0 0 0" rpy="0 0 0"/>
-      <geometry><mesh filename="${head_top_mesh_3}"/></geometry>
-    </collision>
-  </link>
-  <!-- Group left -->
-  <joint name="group_left_chassis_joint_mesh_10_joint" type="fixed">
-    <parent link="base_link"/>
-    <child  link="group_left_chassis_joint_mesh_10_link"/>
-    <origin xyz="0 0 0.112" rpy="0 0 0"/>
-    <limit lower="0" upper="0" effort="0" velocity="1.0"/>
-  </joint>
-  <link name="group_left_chassis_joint_mesh_10_link">
-    <visual>
-      <origin xyz="0 0 0" rpy="0 0 0"/>
-      <geometry>
-        <mesh filename="${group_left_chassis_joint_mesh_10}" scale="${scale_x} ${scale_y} ${scale_z}"/>
-      </geometry>
-      <material name="group_left_chassis_material"/>
-    </visual>
-    <collision>
-      <origin xyz="0 0 0" rpy="0 0 0"/>
-      <geometry><mesh filename="${group_left_chassis_joint_mesh_10}"/></geometry>
-    </collision>
-  </link>
-  <joint name="roup_left_front_suspension_mesh_11_joint" type="fixed">
-    <parent link="group_left_chassis_joint_mesh_10_link"/>
-    <child  link="group_left_front_suspension_mesh_11_link"/>
-    <origin xyz="0.27 0.2 -0.33" rpy="0 0 0"/>
-    <limit lower="0" upper="0" effort="0" velocity="1.0"/>
-  </joint>
-  <link name="group_left_front_suspension_mesh_11_link">
-    <visual>
-      <origin xyz="0 0 0" rpy="0 0 0"/>
-      <geometry>
-        <mesh filename="${group_left_front_suspension_mesh_11}" scale="${scale_x} ${scale_y} ${scale_z}"/>
-      </geometry>
-      <material name="group_left_chassis_material"/>
-    </visual>
-    <collision>
-      <origin xyz="0 0 0" rpy="0 0 0"/>
-      <geometry><mesh filename="${group_left_front_suspension_mesh_11}"/></geometry>
-    </collision>
-  </link>
-  <joint name="group_left_front_steering_mesh_12_joint" type="fixed">
-    <parent link="group_left_front_suspension_mesh_11_link"/>
-    <child  link="group_left_front_steering_mesh_12_link"/>
-    <origin xyz="0.135 0.014 -0.105" rpy="0 0 0"/>
-    <limit lower="0" upper="0" effort="0" velocity="1.0"/>
-  </joint>
-  <link name="group_left_front_steering_mesh_12_link">
-    <visual>
-      <origin xyz="0 0 0" rpy="0 0 0"/>
-      <geometry>
-        <mesh filename="${group_left_front_steering_mesh_12}" scale="${scale_x} ${scale_y} ${scale_z}"/>
-      </geometry>
-      <material name="group_left_front_steering_material"/>
-    </visual>
-    <collision>
-      <origin xyz="0 0 0" rpy="0 0 0"/>
-      <geometry><mesh filename="${group_left_front_steering_mesh_12}"/></geometry>
-    </collision>
-  </link>
-  <joint name="group_left_front_wheel_mesh_13_joint" type="fixed">
-    <parent link="group_left_front_steering_mesh_12_link"/>
-    <child  link="group_left_front_wheel_mesh_13_link"/>
-    <origin xyz="0 0.07 0" rpy="0 0 0"/>
-    <limit lower="0" upper="0" effort="0" velocity="1.0"/>
-  </joint>
-  <link name="group_left_front_wheel_mesh_13_link">
-    <visual>
-      <origin xyz="0 0 0" rpy="0 0 0"/>
-      <geometry>
-        <mesh filename="${group_left_front_wheel_mesh_13}" scale="${scale_x} ${scale_y} ${scale_z}"/>
-      </geometry>
-      <material name="group_left_wheel_material"/>
-    </visual>
-    <collision>
-      <origin xyz="0 0 0" rpy="0 0 0"/>
-      <geometry><mesh filename="${group_left_front_wheel_mesh_13}"/></geometry>
-    </collision>
-  </link>
-<joint name="group_left_middle_suspension_mesh_14_joint" type="fixed">
-    <parent link="group_left_chassis_joint_mesh_10_link"/>
-    <child  link="group_left_middle_suspension_mesh_14_link"/>
-    <origin xyz="0 0 0" rpy="0 0 0"/>
-    <limit lower="0" upper="0" effort="0" velocity="1.0"/>
-  </joint>
-  <link name="group_left_middle_suspension_mesh_14_link">
-    <visual>
-      <origin xyz="0 0 0" rpy="0 0 0"/>
-      <geometry>
-        <mesh filename="${group_left_middle_suspension_mesh_14}" scale="${scale_x} ${scale_y} ${scale_z}"/>
-      </geometry>
-      <material name="group_left_middle_suspension_material"/>
-    </visual>
-    <collision>
-      <origin xyz="0 0 0" rpy="0 0 0"/>
-      <geometry><mesh filename="${group_left_middle_suspension_mesh_14}"/></geometry>
-    </collision>
-  </link>
-<joint name="group_left_middle_chariot_joint_mesh_15_joint" type="fixed">
-    <parent link="group_left_middle_suspension_mesh_14_link"/>
-    <child  link="group_left_middle_chariot_joint_mesh_15_link"/>
-    <origin xyz="-0.175 0.19 -0.32" rpy="0 0 0"/>
-    <limit lower="0" upper="0" effort="0" velocity="1.0"/>
-  </joint>
-  <link name="group_left_middle_chariot_joint_mesh_15_link">
-    <visual>
-      <origin xyz="0 0 0" rpy="0 0 0"/>
-      <geometry>
-        <mesh filename="${group_left_middle_chariot_joint_mesh_15}" scale="${scale_x} ${scale_y} ${scale_z}"/>
-      </geometry>
-      <material name="group_left_middle_chariot_material"/>
-    </visual>
-    <collision>
-      <origin xyz="0 0 0" rpy="0 0 0"/>
-      <geometry><mesh filename="${group_left_middle_chariot_joint_mesh_15}"/></geometry>
-    </collision>
-  </link>
-<joint name="group_left_middle_chariot_center_mesh_16_joint" type="fixed">
-    <parent link="group_left_middle_chariot_joint_mesh_15_link"/>
-    <child  link="group_left_middle_chariot_center_mesh_16_link"/>
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